Commit message: Added materials

File: robot_description/urdf/carriage.urdf.xacro (robot description, xacro)
@@ -14,4 +14,7 @@
                     <mesh filename="package://robot_description/meshes/Carriage.STL"/>
                 </geometry>
+                <material name="purple">
+                    <color rgba="0.7 0.7 1.0 1.0"/>
+                </material>
             </visual>
             <collision>

File: robot_description/urdf/robot.urdf.xacro (robot description, xacro)
@@ -14,4 +14,7 @@
                     <mesh filename="package://robot_description/meshes/Robot_Pan.STL"/>
                 </geometry>
+                <material name="dark_purple">
+                    <color rgba="0.7 0 0.7 1.0"/>
+                </material>
             </visual>
             <collision>
@@ -33,4 +36,7 @@
                     <mesh filename="package://robot_description/meshes/Robot_Arm.STL"/>
                 </geometry>
+                <material name="green">
+                    <color rgba="0.7 1 0.4 1.0"/>
+                </material>
             </visual>
             <collision>
@@ -52,4 +58,7 @@
                     <mesh filename="package://robot_description/meshes/Robot_Forearm.STL"/>
                 </geometry>
+                <material name="blue">
+                    <color rgba="0.4 0.4 1.0 1.0"/>
+                </material>
             </visual>
             <collision>

File: robot_description/urdf/test_robot.urdf.xacro (robot description, xacro)
@@ -12,4 +12,7 @@
                 <mesh filename="package://robot_description/meshes/Base.STL"/>
             </geometry>
+            <material name="light_green">
+                <color rgba="1 0.7 0.7 1.0"/>
+            </material>
         </visual>
         <collision>

Commit message: Adding hardware interface

File: robot_description/urdf/carriage.urdf.xacro (robot description, xacro)
@@ -24,4 +24,13 @@
             </collision>
         </link>
+        <transmission name="carriage_trans">
+            <type>transmission_interface/SimpleTransmission</type>
+            <joint name="carriage_joint">
+                <hardwareInterface>hardware_interface/PositionJointInterface</hardwareInterface>
+            </joint>
+            <actuator name="carriage_motor">
+                <mechanicalReduction>1</mechanicalReduction>
+            </actuator>
+        </transmission>
     </xacro:macro>
 </robot>

File: robot_description/urdf/test_robot.urdf.xacro (robot description, xacro)
@@ -1,4 +1,5 @@
 <?xml version="1.0"?>
 <robot xmlns:xacro="http://ros.org/wiki/xacro" name="test_robot">
+    <xacro:include filename="$(find robot_description)/urdf/gazebo.xacro" />
     <link name="world"/>
     <joint name="base_joint" type="fixed">

Commit message: First working version of gazebo sim

File: robot_description/urdf/carriage.urdf.xacro (robot description, xacro)
@@ -2,11 +2,27 @@
 <robot xmlns:xacro="http://ros.org/wiki/xacro">
     <xacro:macro name="carriage">
-        <joint name="carriage_joint" type="prismatic">
-            <origin xyz="0 0.06 0" rpy="0 ${0.5*pi} 0 "/>
-            <parent link="base_link"/>
-            <child link="carriage_link"/>
-            <limit effort="150.0" lower="-0.3" upper="0.3" velocity="0.5"/>
-            <axis xyz="0 0 1"/>
-        </joint>
+        <link name="base_link">
+            <visual>
+                <geometry>
+                    <mesh filename="package://robot_description/meshes/Base.STL"/>
+                </geometry>
+                <material name="light_green">
+                    <color rgba="1 0.7 0.7 1.0"/>
+                </material>
+            </visual>
+            <collision>
+                <geometry>
+                    <mesh filename="package://robot_description/meshes/Base.STL"/>
+                </geometry>
+            </collision>
+            <inertial>
+                <origin xyz="0 0 0" rpy="0 0 0" />
+                <mass value="1" />
+                <inertia
+                        ixx="1.0" ixy="0.0" ixz="0.0"
+                        iyy="1.0" iyz="0.0"
+                        izz="1.0" />
+            </inertial>
+        </link>
         <link name="carriage_link">
             <visual>
@@ -23,5 +39,20 @@
                 </geometry>
             </collision>
+            <inertial>
+                <origin xyz="0 0 0" rpy="0 0 0" />
+                <mass value="1" />
+                <inertia
+                        ixx="1.0" ixy="0.0" ixz="0.0"
+                        iyy="1.0" iyz="0.0"
+                        izz="1.0" />
+            </inertial>
         </link>
+        <joint name="carriage_joint" type="prismatic">
+            <origin xyz="0 0.06 0" rpy="0 ${0.5*pi} 0 "/>
+            <parent link="base_link"/>
+            <child link="carriage_link"/>
+            <limit effort="150.0" lower="-0.3" upper="0.3" velocity="0.5"/>
+            <axis xyz="0 0 1"/>
+        </joint>
         <transmission name="carriage_trans">
             <type>transmission_interface/SimpleTransmission</type>
@@ -29,8 +60,12 @@
                 <hardwareInterface>hardware_interface/PositionJointInterface</hardwareInterface>
             </joint>
-            <actuator name="carriage_motor">
+            <actuator name="carriage_joint_motor">
+                <hardwareInterface>hardware_interface/PositionJointInterface</hardwareInterface>
                 <mechanicalReduction>1</mechanicalReduction>
             </actuator>
         </transmission>
+        <gazebo reference="carriage_link">
+            <selfCollide>true</selfCollide>
+        </gazebo>
     </xacro:macro>
 </robot>

File: robot_description/urdf/robot.urdf.xacro (robot description, xacro)
@@ -23,5 +23,26 @@
                 </geometry>
             </collision>
+            <inertial>
+                <origin xyz="0 0 0" rpy="0 0 0" />
+                <mass value="1" />
+                <inertia
+                        ixx="1.0" ixy="0.0" ixz="0.0"
+                        iyy="1.0" iyz="0.0"
+                        izz="1.0" />
+            </inertial>
         </link>
+        <transmission name="robot_base_trans">
+            <type>transmission_interface/SimpleTransmission</type>
+            <joint name="robot_base_joint">
+                <hardwareInterface>hardware_interface/PositionJointInterface</hardwareInterface>
+            </joint>
+            <actuator name="robot_base_motor">
+                <hardwareInterface>hardware_interface/PositionJointInterface</hardwareInterface>
+                <mechanicalReduction>1</mechanicalReduction>
+            </actuator>
+        </transmission>
+        <gazebo reference="robot_base_link">
+            <selfCollide>true</selfCollide>
+        </gazebo>
         <joint name="robot_arm_joint" type="revolute">
             <axis xyz="0 0 1"/>
@@ -45,5 +66,26 @@
                 </geometry>
             </collision>
+            <inertial>
+                <origin xyz="0 0 0" rpy="0 0 0" />
+                <mass value="1" />
+                <inertia
+                        ixx="1.0" ixy="0.0" ixz="0.0"
+                        iyy="1.0" iyz="0.0"
+                        izz="1.0" />
+            </inertial>
         </link>
+        <transmission name="robot_arm_trans">
+            <type>transmission_interface/SimpleTransmission</type>
+            <joint name="robot_arm_joint">
+                <hardwareInterface>hardware_interface/PositionJointInterface</hardwareInterface>
+            </joint>
+            <actuator name="robot_arm_motor">
+                <hardwareInterface>hardware_interface/PositionJointInterface</hardwareInterface>
+                <mechanicalReduction>1</mechanicalReduction>
+            </actuator>
+        </transmission>
+        <gazebo reference="robot_arm_link">
+            <selfCollide>true</selfCollide>
+        </gazebo>
         <joint name="robot_forearm_joint" type="revolute">
             <axis xyz="0 0 1"/>
@@ -67,5 +109,26 @@
                 </geometry>
             </collision>
+            <inertial>
+                <origin xyz="0 0 0" rpy="0 0 0" />
+                <mass value="1" />
+                <inertia
+                        ixx="1.0" ixy="0.0" ixz="0.0"
+                        iyy="1.0" iyz="0.0"
+                        izz="1.0" />
+            </inertial>
         </link>
+        <transmission name="robot_forearm_trans">
+            <type>transmission_interface/SimpleTransmission</type>
+            <joint name="robot_forearm_joint">
+                <hardwareInterface>hardware_interface/PositionJointInterface</hardwareInterface>
+            </joint>
+            <actuator name="robot_forearm_motor">
+                <hardwareInterface>hardware_interface/PositionJointInterface</hardwareInterface>
+                <mechanicalReduction>1</mechanicalReduction>
+            </actuator>
+        </transmission>
+        <gazebo reference="robot_forearm_link">
+            <selfCollide>true</selfCollide>
+        </gazebo>
         <joint name="robot_wrist_joint" type="revolute">
             <axis xyz="0 1 0"/>
@@ -86,5 +149,26 @@
                 </geometry>
             </collision>
+            <inertial>
+                <origin xyz="0 0 0" rpy="0 0 0" />
+                <mass value="1" />
+                <inertia
+                        ixx="1.0" ixy="0.0" ixz="0.0"
+                        iyy="1.0" iyz="0.0"
+                        izz="1.0" />
+            </inertial>
         </link>
+        <transmission name="robot_wrist_trans">
+            <type>transmission_interface/SimpleTransmission</type>
+            <joint name="robot_wrist_joint">
+                <hardwareInterface>hardware_interface/PositionJointInterface</hardwareInterface>
+            </joint>
+            <actuator name="robot_wrist_motor">
+                <hardwareInterface>hardware_interface/PositionJointInterface</hardwareInterface>
+                <mechanicalReduction>1</mechanicalReduction>
+            </actuator>
+        </transmission>
+        <gazebo reference="robot_wrist_link">
+            <selfCollide>true</selfCollide>
+        </gazebo>
         <joint name="end_effector" type="fixed">
             <origin xyz="0 0.035 0" rpy="0 0 0"/>

File: robot_description/urdf/test_robot.urdf.xacro (robot description, xacro)
@@ -1,5 +1,9 @@
 <?xml version="1.0"?>
 <robot xmlns:xacro="http://ros.org/wiki/xacro" name="test_robot">
-    <xacro:include filename="$(find robot_description)/urdf/gazebo.xacro" />
+    <xacro:include filename="$(find robot_description)/urdf/gazebo_plugins.xacro"/>
+    <xacro:include filename="$(find robot_description)/urdf/carriage.urdf.xacro"/>
+    <xacro:include filename="$(find robot_description)/urdf/robot.urdf.xacro"/>
+    <xacro:carriage/>
+    <xacro:robot/>
     <link name="world"/>
     <joint name="base_joint" type="fixed">
@@ -8,22 +12,3 @@
         <child link="base_link"/>
     </joint>
-    <link name="base_link">
-        <visual>
-            <geometry>
-                <mesh filename="package://robot_description/meshes/Base.STL"/>
-            </geometry>
-            <material name="light_green">
-                <color rgba="1 0.7 0.7 1.0"/>
-            </material>
-        </visual>
-        <collision>
-            <geometry>
-                <mesh filename="package://robot_description/meshes/Base.STL"/>
-            </geometry>
-        </collision>
-    </link>
-    <xacro:include filename="$(find robot_description)/urdf/carriage.urdf.xacro"/>
-    <xacro:carriage/>
-        <xacro:include filename="$(find robot_description)/urdf/robot.urdf.xacro"/>
-        <xacro:robot/>
 </robot>
